File: Eagle Files/AbbotCameraController.brd (EAGLE design)
At the start: 165.1 x 74.6 mm, 80 parts, among them IC1 7805TV, J1 AVR_SPI_PRG_6NS, J2 POWER_JACKPTH_LOCK, Q1 2N3904, Q10 2N3904, Q11 2N3904, Q12 2N3904, Q2 2N3904, Q3 2N3904, Q4 2N3904, Q5 2N3904, Q6 2N3904, Q7 2N3904, Q8 2N3904, Q9 2N3904, U1 ATMEGA328P_PDIP, Y1 16MHz

Commit message: Eagle Files To Be Fabricated
Added Ultrasound Breakout, Load Cell Breakout, Aux Breakout, Resistors
to Switches.  Changed Arduino Profile.
Parts:
- removed U1: ATMEGA328P_PDIP, SparkFun-DigitalIC:DIL28-3
- added IC2: MCP23017SP, adafruit:DIL28-3
- added JP5: (no value), SparkFun-Connectors:1X04_LONGPADS
- added JP6, JP7, JP8, JP9: (no value), SparkFun-Connectors:1X03_LONGPADS
- added LED14, LED15, LED16, LED17: (no value), SparkFun-LED:LED5MM
- added Q13, Q14, Q15, Q16: 2N3904, transistor-npn:TO92
- added R15, R16, R17, R18, R19, R20, R21, R22, R23, R24, R25, R26, R30, R32, R34, R36: 1k, rcl:0207/10
- added R27, R28: 4.7k, rcl:0207/10
- added R29: 10, rcl:0207/10
- added R31, R33, R35, R37: 10k, rcl:0207/10
- added R38, R39, R40, R41: 220, rcl:0207/10
- added U$1: INA125P, EzerLonginus:16-DIP
- added U14: ATMEGA328P, SparkFun-DigitalIC:TQFP32-08
- JP2, JP3, JP4: device SparkFun-Connectors:1X06 -> SparkFun-Connectors:1X04
- R1, R10, R11, R12, R2, R3, R4, R5, R6, R7, R8, R9: value 1k -> 220
- moved JP3 152.5 mm to (157.5, 57.1), turned to 90 degrees
- moved JP2 150.0 mm to (160.0, 57.1)
- moved JP4 147.5 mm to (154.9, 57.1), turned to 90 degrees
- moved J1 81.2 mm to (97.8, 82.5), turned to 180 degrees
- moved JP1 50.2 mm to (81.3, 83.8)
- moved C6 23.4 mm to (64.8, 83.8), turned to 180 degrees
- moved LED13 21.0 mm to (119.4, 82.5)
- moved D1 15.2 mm to (130.8, 78.7)
- moved IC1 14.0 mm to (130.8, 81.3)
- moved C4 12.8 mm to (128.3, 69.8)
- moved J2 12.7 mm to (147.3, 91.4)
- moved C3 12.7 mm to (137.2, 69.8)
- moved C5 12.7 mm to (123.2, 69.8)
- moved C1 12.6 mm to (72.4, 63.5)
- moved Y1 12.6 mm to (81.3, 64.8)
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Connections:
- new net A00: JP6.2, U14.23
- new net A01: JP7.2, U14.24
- new net A02: JP8.2, U14.25
- new net A03: JP9.2, U14.26
- new net A06: U$1.10, U$1.11, U14.19
- new net A07: U14.22
- new net AREF: JP1.P$5, U14.20
- new net CAM1: IC2.21, Q1.2, R15.1
- new net CAM10: IC2.2, Q10.2, R24.1
- new net CAM11: IC2.3, Q11.2, R25.1
- new net CAM12: IC2.4, Q12.2, R26.1
- new net CAM2: IC2.22, Q2.2, R16.1
- new net CAM3: IC2.23, Q3.2, R17.1
- new net CAM4: IC2.24, Q4.2, R18.1
- new net CAM5: IC2.25, Q5.2, R19.1
- new net CAM6: IC2.26, Q6.2, R20.1
- new net CAM7: IC2.27, Q7.2, R21.1
- new net CAM8: IC2.28, Q8.2, R22.1
- new net CAM9: IC2.1, Q9.2, R23.1
- new net D02: R30.2
- new net D03: R32.2
- new net D04: R34.2
- new net D05: R36.2
- new net N$35: R15.2, S1.1
- new net N$36: R16.2, S2.1
- new net N$41: R17.2, S3.1
- new net N$42: R18.2, S4.1
- new net N$43: R19.2, S5.1
- new net N$44: R20.2, S6.1
- new net N$45: R21.2, S7.1
- new net N$46: R22.2, S8.1
- new net N$47: R23.2, S9.1
- new net N$48: R24.2, S10.1
- new net N$49: R25.2, S11.1
- new net N$50: R26.2, S12.1
- new net N$51: U$1.15, U$1.4
- new net N$52: JP5.1, U$1.7
- new net N$53: R29.1, U$1.9
- new net N$54: Q15.2, R34.1, R35.1
- new net N$55: JP8.3, LED16.K, Q15.1
- new net N$56: Q16.2, R36.1, R37.1
- new net N$57: JP9.3, LED17.K, Q16.1
- new net N$58: LED14.A, R38.2
- new net N$59: LED15.A, R39.2
- new net N$60: LED16.A, R40.2
- new net N$62: LED17.A, R41.2
- new net SCL: IC2.12, R27.1, U14.28
- new net SDA: IC2.13, R28.1, U14.27
- net +5V: now also IC2.18, IC2.9, JP2.1, JP2.2, JP2.3, JP2.4, JP5.4, JP6.1, JP7.1, JP8.1, JP9.1, R27.2, R28.2, R38.1, R39.1, R40.1, R41.1, U$1.1, U$1.2, U14.18, U14.4, U14.6; no longer JP3.1, JP3.2, JP3.3, JP3.4, JP3.5, JP3.6, U1.20, U1.21, U1.7
- net D10: now also U14.14; no longer Q9.2, S9.1, U1.16
- net D11: now also U14.15; no longer Q10.2, S10.1, U1.17
- net D12: now also U14.16; no longer Q11.2, S11.1, U1.18
- net D13: now also U14.17; no longer Q12.2, S12.1, U1.19
- net D2: now also U14.32; no longer Q1.2, S1.1, U1.4
- net D3: now also U14.1; no longer Q2.2, S2.1, U1.5
- net D4: now also U14.2; no longer Q3.2, S3.1, U1.6
- net D5: now also U14.9; no longer Q4.2, S4.1, U1.11
- net D6: now also JP3.1, U14.10; no longer Q5.2, S5.1, U1.12
- net D7: now also JP3.2, U14.11; no longer Q6.2, S6.1, U1.13
- net D8: now also JP3.3, U14.12; no longer Q7.2, S7.1, U1.14
- net D9: now also JP3.4, U14.13; no longer Q8.2, S8.1, U1.15
- net GND: now also IC2.10, IC2.15, IC2.16, IC2.17, JP5.3, Q13.3, Q14.3, Q15.3, Q16.3, R31.2, R33.2, R35.2, R37.2, U$1.12, U$1.3, U$1.5, U14.21, U14.3, U14.5; no longer JP1.P$5, JP4.5, JP4.6, U1.22, U1.8
- net N$25: now also Q13.2, R30.1, R31.1; no longer JP2.1, U1.23
- net N$27: now also Q14.2, R32.1, R33.1; no longer JP2.2, U1.24
- net N$28: now also JP6.3, LED14.K, Q13.1; no longer JP2.3, U1.25
- net N$29: now also JP7.3, LED15.K, Q14.1; no longer JP2.4, U1.26
- net N$30: now also U14.7; no longer U1.9
- net N$31: now also U14.8; no longer U1.10
- net N$33: now also JP5.2, U$1.6; no longer JP2.5, U1.27
- net N$34: now also R29.2, U$1.8; no longer JP2.6, U1.28
- net RST: now also U14.29; no longer U1.1
- net RXI: now also U14.30; no longer U1.2
- net TXO: now also U14.31; no longer U1.3
Routing:
- net +5V: track 410.7 -> 594.0 mm
- net D13: track 198.5 -> 17.6 mm
- net D11: track 179.3 -> 16.3 mm, vias 0 -> 1
- net D12: track 169.7 -> 23.3 mm, vias 1 -> 0
- net CAM12: track 0.00 -> 109.8 mm
- net CAM1: track 0.00 -> 99.1 mm
- net CAM11: track 0.00 -> 96.9 mm
- net D2: track 93.2 -> 0.00 mm
- net N$25: track 107.4 -> 14.6 mm
- net CAM2: track 0.00 -> 88.9 mm
- net CAM3: track 0.00 -> 87.6 mm
- net D3: track 84.4 -> 0.00 mm
- net D5: track 80.8 -> 0.00 mm
- net D10: track 79.8 -> 0.00 mm
- net A03: track 0.00 -> 75.2 mm, vias 0 -> 1
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Other:
- board size 165.1 x 74.6 mm -> 165.1 x 88.6 mm
- board text added: "+5V"
- board text added: "0.1uF"
- board text added: "10"
- board text added: "100uF"
- board text added: "10k"
- board text added: "10uF"
- board text added: "16MHz"
- board text added: "1N4001"
- board text added: "1k"
- board text added: "220"
- board text added: "22pF"
- board text added: "2N3904"
- board text added: "4k7"
- board text added: "7805"
- board text added: "ATMEGA328"
- board text added: "Abbott Camera Controller"
- board text added: "C1"
- board text added: "C2"
- board text added: "C3"
- board text added: "C4"
- board text added: "C5"
- board text added: "C6"
- board text added: "D06"
- board text added: "D07"
- board text added: "D08"
- board text added: "D09"
- board text added: "D1"
- board text added: "E+"
- board text added: "E-"
- board text added: "GND"
- board text added: "GPIO"
- board text added: "INA125P"
- board text added: "LED1"
- board text added: "LED10"
- board text added: "LED11"
- board text added: "LED12"
- board text added: "LED13"
- board text added: "LED14"
- board text added: "LED15"
- board text added: "LED16"
- board text added: "LED17"
- board text added: "LED2"
- board text added: "LED3"
- board text added: "LED4"
- board text added: "LED5"
- board text added: "LED6"
- board text added: "LED7"
- board text added: "LED8"
- board text added: "LED9"
- board text added: "LOAD CELL"
- board text added: "MCP23017SP"
- board text added: "MISO"
- board text added: "MOSI"
- board text added: "March 2014"
- board text added: "Q1"
- board text added: "Q10"
- board text added: "Q11"
- board text added: "Q12"
- board text added: "Q13"
- board text added: "Q14"
- board text added: "Q15"
- board text added: "Q16"
- board text added: "Q2"
- board text added: "Q3"
- board text added: "Q4"
- board text added: "Q5"
- board text added: "Q6"
- board text added: "Q7"
- board text added: "Q8"
- board text added: "Q9"
- board text added: "R1"
- board text added: "R10"
- board text added: "R11"
- board text added: "R12"
- board text added: "R13"
- board text added: "R14"
- board text added: "R15"
- board text added: "R16"
- board text added: "R17"
- board text added: "R18"
- board text added: "R19"
- board text added: "R2"
- board text added: "R20"
- board text added: "R21"
- board text added: "R22"
- board text added: "R23"
- board text added: "R24"
- board text added: "R25"
- board text added: "R26"
- board text added: "R27"
- board text added: "R28"
- board text added: "R29"
- board text added: "R3"
- board text added: "R30"
- board text added: "R31"
- board text added: "R32"
- board text added: "R33"
- board text added: "R34"
- board text added: "R35"
- board text added: "R36"
- board text added: "R37"
- board text added: "R38"
- board text added: "R39"
- board text added: "R4"
- board text added: "R40"
- board text added: "R41"
- board text added: "R5"
- board text added: "R6"
- board text added: "R7"
- board text added: "R8"
- board text added: "R9"
- board text added: "RST"
- board text added: "S+"
- board text added: "S-"
- board text added: "S01"
- board text added: "S02"
- board text added: "S03"
- board text added: "S04"
- board text added: "SCK"
- board text added: "Version 01"

Commit message: Initial Arduino Code
Uploaded some test code for Arduino.  It
Connections:
- removed net D2: U14.32
- removed net D3: U14.1
- removed net D4: U14.2
- removed net D5: U14.9
- net D02: now also U14.32
- net D03: now also U14.1
- net D04: now also U14.2
- net D05: now also U14.9
Routing:
- net D05: track 0.00 -> 92.8 mm, vias 0 -> 1
- net D04: track 0.00 -> 48.5 mm, vias 0 -> 1
- net D03: track 0.00 -> 36.3 mm, vias 0 -> 1
- net D02: track 0.00 -> 22.2 mm, vias 0 -> 1
Changed lines of the file:
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@@
 <via x="80.264" y="72.644" extent="1-16" drill="0.6096" shape="octagon"/>
-</signal>
-<signal name="D2">
-<contactref element="U14" pad="32"/>
-</signal>
-<signal name="D3">
-<contactref element="U14" pad="1"/>
-</signal>
-<signal name="D4">
-<contactref element="U14" pad="2"/>
-</signal>
-<signal name="D5">
-<contactref element="U14" pad="9"/>
 </signal>
 <signal name="D6">
@@
 <signal name="D02">
 <contactref element="R30" pad="2"/>
+<contactref element="U14" pad="32"/>
+<wire x1="74.676" y1="76.2" x2="76.2" y2="76.2" width="0.254" layer="1"/>
+<wire x1="74.168" y1="75.692" x2="74.676" y2="76.2" width="0.254" layer="16"/>
+<wire x1="70.612" y1="75.692" x2="74.168" y2="75.692" width="0.254" layer="16"/>
+<wire x1="68.072" y1="73.152" x2="70.612" y2="75.692" width="0.254" layer="16"/>
+<wire x1="61.468" y1="73.152" x2="68.072" y2="73.152" width="0.254" layer="16"/>
+<wire x1="57.404" y1="69.088" x2="61.468" y2="73.152" width="0.254" layer="16"/>
+<wire x1="76.2" y1="76.2" x2="76.264771875" y2="75.985425" width="0.254" layer="1"/>
+<wire x1="57.404" y1="69.088" x2="57.15" y2="69.088" width="0.254" layer="16"/>
+<via x="74.676" y="76.2" extent="1-16" drill="0.6096" shape="octagon"/>
 </signal>
 <signal name="N$28">
@@
 <signal name="D03">
 <contactref element="R32" pad="2"/>
+<contactref element="U14" pad="1"/>
+<wire x1="75.184" y1="74.168" x2="76.2" y2="74.168" width="0.254" layer="1"/>
+<wire x1="72.644" y1="76.708" x2="75.184" y2="74.168" width="0.254" layer="1"/>
+<wire x1="72.136" y1="76.2" x2="72.644" y2="76.708" width="0.254" layer="16"/>
+<wire x1="70.104" y1="76.2" x2="72.136" y2="76.2" width="0.254" layer="16"/>
+<wire x1="67.564" y1="73.66" x2="70.104" y2="76.2" width="0.254" layer="16"/>
+<wire x1="59.944" y1="73.66" x2="67.564" y2="73.66" width="0.254" layer="16"/>
+<wire x1="56.388" y1="70.104" x2="59.944" y2="73.66" width="0.254" layer="16"/>
+<wire x1="45.72" y1="70.104" x2="56.388" y2="70.104" width="0.254" layer="16"/>
+<wire x1="44.704" y1="69.088" x2="45.72" y2="70.104" width="0.254" layer="16"/>
+<wire x1="76.2" y1="74.168" x2="76.264771875" y2="73.874571875" width="0.254" layer="1"/>
+<wire x1="44.704" y1="69.088" x2="44.45" y2="69.088" width="0.254" layer="16"/>
+<via x="72.644" y="76.708" extent="1-16" drill="0.6096" shape="octagon"/>
 </signal>
 <signal name="N$54">
@@
 <signal name="D04">
 <contactref element="R34" pad="2"/>
+<contactref element="U14" pad="2"/>
+<wire x1="76.2" y1="72.644" x2="76.708" y2="73.152" width="0.254" layer="1"/>
+<wire x1="75.184" y1="72.644" x2="76.2" y2="72.644" width="0.254" layer="1"/>
+<wire x1="72.644" y1="70.104" x2="75.184" y2="72.644" width="0.254" layer="16"/>
+<wire x1="59.944" y1="70.104" x2="72.644" y2="70.104" width="0.254" layer="16"/>
+<wire x1="57.912" y1="68.072" x2="59.944" y2="70.104" width="0.254" layer="16"/>
+<wire x1="37.084" y1="68.072" x2="57.912" y2="68.072" width="0.254" layer="16"/>
+<wire x1="35.052" y1="70.104" x2="37.084" y2="68.072" width="0.254" layer="16"/>
+<wire x1="33.02" y1="70.104" x2="35.052" y2="70.104" width="0.254" layer="16"/>
+<wire x1="32.004" y1="69.088" x2="33.02" y2="70.104" width="0.254" layer="16"/>
+<wire x1="76.708" y1="73.152" x2="76.830459375" y2="73.308884375" width="0.254" layer="1"/>
+<wire x1="32.004" y1="69.088" x2="31.75" y2="69.088" width="0.254" layer="16"/>
+<via x="75.184" y="72.644" extent="1-16" drill="0.6096" shape="octagon"/>
 </signal>
 <signal name="D05">
 <contactref element="R36" pad="2"/>
+<contactref element="U14" pad="9"/>
+<wire x1="85.344" y1="67.056" x2="82.804" y2="69.596" width="0.254" layer="1"/>
+<wire x1="85.344" y1="56.388" x2="85.344" y2="67.056" width="0.254" layer="1"/>
+<wire x1="84.836" y1="55.88" x2="85.344" y2="56.388" width="0.254" layer="16"/>
+<wire x1="37.592" y1="55.88" x2="84.836" y2="55.88" width="0.254" layer="16"/>
+<wire x1="35.56" y1="57.912" x2="37.592" y2="55.88" width="0.254" layer="16"/>
+<wire x1="35.56" y1="68.072" x2="35.56" y2="57.912" width="0.254" layer="16"/>
+<wire x1="20.32" y1="68.072" x2="35.56" y2="68.072" width="0.254" layer="16"/>
+<wire x1="19.304" y1="69.088" x2="20.32" y2="68.072" width="0.254" layer="16"/>
+<wire x1="82.804" y1="69.596" x2="82.335425" y2="69.914771875" width="0.254" layer="1"/>
+<wire x1="19.304" y1="69.088" x2="19.05" y2="69.088" width="0.254" layer="16"/>
+<via x="85.344" y="56.388" extent="1-16" drill="0.6096" shape="octagon"/>
 </signal>
 <signal name="N$58">
