File: Eagle Files/AbbotCameraController.sch (EAGLE design)
At the start: 80 parts, among them IC1 7805TV, J1 AVR_SPI_PRG_6NS, J2 POWER_JACKPTH_LOCK, Q1 2N3904, Q10 2N3904, Q11 2N3904, Q12 2N3904, Q2 2N3904, Q3 2N3904, Q4 2N3904, Q5 2N3904, Q6 2N3904, Q7 2N3904, Q8 2N3904, Q9 2N3904, U1 ATMEGA328P_PDIP, Y1 16MHz

Commit message: Eagle Files To Be Fabricated
Added Ultrasound Breakout, Load Cell Breakout, Aux Breakout, Resistors
to Switches.  Changed Arduino Profile.
Parts:
- removed U1: ATMEGA328P_PDIP, SparkFun-DigitalIC:ATMEGA328P_PDIP
- added IC2: MCP23017SP, adafruit:MCP23017SP
- added JP5: (no value), SparkFun-Connectors:M04LONGPADS
- added JP6, JP7, JP8, JP9: (no value), SparkFun-Connectors:M03LONGPADS
- added LED14, LED15, LED16, LED17: (no value), SparkFun-LED:LED5MM
- added Q13, Q14, Q15, Q16: 2N3904, transistor-npn:2N3904
- added R15, R16, R17, R18, R19, R20, R21, R22, R23, R24, R25, R26, R30, R32, R34, R36: 1k, rcl:R-US_0207/10
- added R27, R28: 4.7k, rcl:R-US_0207/10
- added R29: 10, rcl:R-US_0207/10
- added R31, R33, R35, R37: 10k, rcl:R-US_0207/10
- added R38, R39, R40, R41: 220, rcl:R-US_0207/10
- added U$1: INA125P, EzerLonginus:INA125P
- added U14: ATMEGA328P, SparkFun-DigitalIC:ATMEGA328_SMT
- JP2, JP3, JP4: device SparkFun-Connectors:M06SIP -> SparkFun-Connectors:M04PTH
- R1, R10, R11, R12, R2, R3, R4, R5, R6, R7, R8, R9: value 1k -> 220
Connections:
- new net A00: JP6.2, U14.PC0(ADC0)
- new net A01: JP7.2, U14.PC1(ADC1)
- new net A02: JP8.2, U14.PC2(ADC2)
- new net A03: JP9.2, U14.PC3(ADC3)
- new net A06: U$1.SENSE, U$1.VO, U14.ADC6
- new net A07: U14.ADC7
- new net AREF: JP1.CTS, U14.AREF
- new net CAM1: IC2.GPA0, Q1.B, R15.1
- new net CAM10: IC2.GPB1, Q10.B, R24.1
- new net CAM11: IC2.GPB2, Q11.B, R25.1
- new net CAM12: IC2.GPB3, Q12.B, R26.1
- new net CAM2: IC2.GPA1, Q2.B, R16.1
- new net CAM3: IC2.GPA2, Q3.B, R17.1
- new net CAM4: IC2.GPA3, Q4.B, R18.1
- new net CAM5: IC2.GPA4, Q5.B, R19.1
- new net CAM6: IC2.GPA5, Q6.B, R20.1
- new net CAM7: IC2.GPA6, Q7.B, R21.1
- new net CAM8: IC2.GPA7, Q8.B, R22.1
- new net CAM9: IC2.GPB0, Q9.B, R23.1
- new net D02: R30.2
- new net D03: R32.2
- new net D04: R34.2
- new net D05: R36.2
- new net N$35: R15.2, S1.1
- new net N$36: R16.2, S2.1
- new net N$41: R17.2, S3.1
- new net N$42: R18.2, S4.1
- new net N$43: R19.2, S5.1
- new net N$44: R20.2, S6.1
- new net N$45: R21.2, S7.1
- new net N$46: R22.2, S8.1
- new net N$47: R23.2, S9.1
- new net N$48: R24.2, S10.1
- new net N$49: R25.2, S11.1
- new net N$50: R26.2, S12.1
- new net N$51: U$1.VREF5, U$1.VREFOUT
- new net N$52: JP5.1, U$1.VIN-
- new net N$53: R29.1, U$1.RG2
- new net N$54: Q15.B, R34.1, R35.1
- new net N$55: JP8.3, LED16.C, Q15.C
- new net N$56: Q16.B, R36.1, R37.1
- new net N$57: JP9.3, LED17.C, Q16.C
- new net N$58: LED14.A, R38.2
- new net N$59: LED15.A, R39.2
- new net N$60: LED16.A, R40.2
- new net N$62: LED17.A, R41.2
- new net SCL: IC2.SCL, R27.1, U14.PC5(ADC5/SCL)
- new net SDA: IC2.SDA, R28.1, U14.PC4(ADC4/SDA)
- net +5V: now also IC2.!RESET, IC2.VDD, JP2.1, JP2.2, JP2.3, JP2.4, JP5.4, JP6.1, JP7.1, JP8.1, JP9.1, R27.2, R28.2, R38.1, R39.1, R40.1, R41.1, U$1.+5V, U$1.SLP, U14.AVCC, U14.VCC@1, U14.VCC@2; no longer JP3.1, JP3.2, JP3.3, JP3.4, JP3.5, JP3.6, U1.AREF, U1.AVCC, U1.VCC
- net D10: now also U14.PB2(SS/OC1B); no longer Q9.B, S9.1, U1.PB2(SS/OC1B)
- net D11: now also U14.PB3(MOSI/OC2); no longer Q10.B, S10.1, U1.PB3(MOSI/OC2)
- net D12: now also U14.PB4(MISO); no longer Q11.B, S11.1, U1.PB4(MISO)
- net D13: now also U14.PB5(SCK); no longer Q12.B, S12.1, U1.PB5(SCK)
- net D2: now also U14.PD2(INT0); no longer Q1.B, S1.1, U1.PD2(INT0)
- net D3: now also U14.PD3(INT1); no longer Q2.B, S2.1, U1.PD3(INT1)
- net D4: now also U14.PD4(XCK/T0); no longer Q3.B, S3.1, U1.PD4(XCK/T0)
- net D5: now also U14.PD5(T1); no longer Q4.B, S4.1, U1.PD5(T1)
- net D6: now also JP3.1, U14.PD6(AIN0); no longer Q5.B, S5.1, U1.PD6(AIN0)
- net D7: now also JP3.2, U14.PD7(AIN1); no longer Q6.B, S6.1, U1.PD7(AIN1)
- net D8: now also JP3.3, U14.PB0(ICP); no longer Q7.B, S7.1, U1.PB0(ICP)
- net D9: now also JP3.4, U14.PB1(OC1A); no longer Q8.B, S8.1, U1.PB1(OC1A)
- net GND: now also IC2.A0, IC2.A1, IC2.A2, IC2.VSS, JP5.3, Q13.E, Q14.E, Q15.E, Q16.E, R31.2, R33.2, R35.2, R37.2, U$1.IAREF, U$1.V-, U$1.VREFCOM, U14.AGND, U14.GND@1, U14.GND@2; no longer JP1.CTS, JP4.5, JP4.6, U1.GND@1, U1.GND@2
- net N$25: now also Q13.B, R30.1, R31.1; no longer JP2.1, U1.PC0(ADC0)
- net N$27: now also Q14.B, R32.1, R33.1; no longer JP2.2, U1.PC1(ADC1)
- net N$28: now also JP6.3, LED14.C, Q13.C; no longer JP2.3, U1.PC2(ADC2)
- net N$29: now also JP7.3, LED15.C, Q14.C; no longer JP2.4, U1.PC3(ADC3)
- net N$30: now also U14.PB6(XTAL1/TOSC1); no longer U1.PB6(XTAL1/TOSC1)
- net N$31: now also U14.PB7(XTAL2/TOSC2); no longer U1.PB7(XTAL2/TOSC2)
- net N$33: now also JP5.2, U$1.VIN+; no longer JP2.5, U1.PC4(ADC4/SDA)
- net N$34: now also R29.2, U$1.RG1; no longer JP2.6, U1.PC5(ADC5/SCL)
- net RST: now also U14.PC6(/RESET); no longer U1.PC6(/RESET)
- net RXI: now also U14.PD0(RXD); no longer U1.PD0(RXD)
- net TXO: now also U14.PD1(TXD); no longer U1.PD1(TXD)
Other:
- note added: "AUX GPIO PINS"
- note added: "DIGITAL OUTPUT EXPANDER"
- note added: "LOAD CELL SESNOR"
- note added: "ULTRASOUND SENSORS"
- note removed: "AUX POWER PINS"
- moved on the sheet: C3, C4, C5, D1, IC1, J1, J2, JP1, LED1, LED10, LED11, LED12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

Commit message: Initial Arduino Code
Uploaded some test code for Arduino.  It
Connections:
- removed net D2: U14.PD2(INT0)
- removed net D3: U14.PD3(INT1)
- removed net D4: U14.PD4(XCK/T0)
- removed net D5: U14.PD5(T1)
- net D02: now also U14.PD2(INT0)
- net D03: now also U14.PD3(INT1)
- net D04: now also U14.PD4(XCK/T0)
- net D05: now also U14.PD5(T1)
Changed lines of the file:
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@@
-</segment>
-</net>
-<net name="D2" class="0">
-<segment>
-<wire x1="269.24" y1="-73.66" x2="274.32" y2="-73.66" width="0.1524" layer="91"/>
-<label x="271.78" y="-73.66" size="1.778" layer="95"/>
-<pinref part="U14" gate="G$1" pin="PD2(INT0)"/>
 </segment>
 </net>
@@
 </segment>
 </net>
-<net name="D3" class="0">
-<segment>
-<wire x1="269.24" y1="-76.2" x2="274.32" y2="-76.2" width="0.1524" layer="91"/>
-<label x="271.78" y="-76.2" size="1.778" layer="95"/>
-<pinref part="U14" gate="G$1" pin="PD3(INT1)"/>
-</segment>
-</net>
-<net name="D4" class="0">
-<segment>
-<wire x1="269.24" y1="-78.74" x2="274.32" y2="-78.74" width="0.1524" layer="91"/>
-<label x="271.78" y="-78.74" size="1.778" layer="95"/>
-<pinref part="U14" gate="G$1" pin="PD4(XCK/T0)"/>
-</segment>
-</net>
-<net name="D5" class="0">
-<segment>
-<wire x1="269.24" y1="-81.28" x2="274.32" y2="-81.28" width="0.1524" layer="91"/>
-<label x="271.78" y="-81.28" size="1.778" layer="95"/>
-<pinref part="U14" gate="G$1" pin="PD5(T1)"/>
-</segment>
-</net>
 <net name="D6" class="0">
 <segment>
@@
 <label x="190.5" y="96.52" size="1.778" layer="95" font="vector"/>
 </segment>
+<segment>
+<wire x1="269.24" y1="-73.66" x2="274.32" y2="-73.66" width="0.1524" layer="91"/>
+<label x="271.78" y="-73.66" size="1.778" layer="95"/>
+<pinref part="U14" gate="G$1" pin="PD2(INT0)"/>
+</segment>
 </net>
 <net name="N$28" class="0">
@@
 <label x="241.3" y="96.52" size="1.778" layer="95" font="vector"/>
 </segment>
+<segment>
+<wire x1="269.24" y1="-76.2" x2="274.32" y2="-76.2" width="0.1524" layer="91"/>
+<label x="271.78" y="-76.2" size="1.778" layer="95"/>
+<pinref part="U14" gate="G$1" pin="PD3(INT1)"/>
+</segment>
 </net>
 <net name="N$54" class="0">
@@
 <label x="292.1" y="96.52" size="1.778" layer="95" font="vector"/>
 </segment>
+<segment>
+<wire x1="269.24" y1="-78.74" x2="274.32" y2="-78.74" width="0.1524" layer="91"/>
+<label x="271.78" y="-78.74" size="1.778" layer="95"/>
+<pinref part="U14" gate="G$1" pin="PD4(XCK/T0)"/>
+</segment>
 </net>
 <net name="D05" class="0">
@@
 <label x="342.9" y="96.52" size="1.778" layer="95" font="vector"/>
 </segment>
-</net>
+<segment>
+<wire x1="269.24" y1="-81.28" x2="274.32" y2="-81.28" width="0.1524" layer="91"/>
+<label x="271.78" y="-81.28" size="1.778" layer="95"/>
+<pinref part="U14" gate="G$1" pin="PD5(T1)"/>
+</segment>
+</net>
